Commit message: update control package name to `ib2_control`

File: int-ball2_control/description/ib2.urdf (robot description, URDF)
Before this commit: robot ib2, 6 links, 5 joints
Links:
- link body: geometry collision mesh filename=package://ib2_control/description/media/meshes/int-ball2/in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; visual mesh filename=package://ib2_control/description/media/meshes/int-ball2/in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
